File: midi-bit-box-v1.sch (EAGLE design)
At the start: 51 parts, among them IC1 LM386, IC2 CD4024BE, T1 42TM011-RC, U1 AY-3-8910

Commit message: Added SPST and latching relay switching circuit
Parts:
- removed SWITCH: (no value), switches:SPDT.WIRE
- added BLAST: SPST, switches:SPST
- added C19: 1uF, caps-film:CAP.4
- added C20: 100uF, caps-elec:5MM.2
- added C3, C4: 100nF, caps-film:CAP.2
- added IC3: 78L09, SamacSys_Parts:L78L09ACZ-TR
- added IC4: NE555, integrated circuits:DIP8_TH
- added IND2: 5MM_LED, diodes:LED.2
- added K1: PANASONIC_TQ2-L-5VPANASONIC_TQ2-L-5V_0_0, Panasonic - TQ2-L-5V:PANASONIC_TQ2-L-5VPANASONIC_TQ2-L-5V_0_0
- added Q1, Q2, Q3: 2N3904, transistors-BJT:2N5088
- added Q4: 2N3906, transistors-BJT:2N5087
- added R1, R2: (no value), resistors:R.3B
- added R17: 100K, resistors:R.3B
- added R18, R19, R21: 10K, resistors:R.3B
- added R20: 4.7K, resistors:R.3B
Connections:
- removed net N$49: R10.2, R11.2, R12.2, R13.2, SWITCH.1
- new net N$40: BLAST.2, C19.2, R17.2
- new net N$50: IND2.A, R20.2
- new net N$51: Q2.C, R21.1
- new net N$52: Q2.B, R18.1
- new net N$53: Q1.B, R19.1
- new net N$54: IND2.C, Q1.C
- new net N$55: C20.+, Q3.E, Q4.E
- new net N$56: Q3.B, Q4.B
- new net N$57: C20.-, K1.S+/R-
- new net N$58: C18.-, K1.2, K1.7, R16.2
- new net N$59: K1.9, R10.2, R11.2, R12.2, R13.2
- new net N$7: IC4.3, R17.1, R18.2, R19.2
- new net VC: C4.1, IC3.VOUT, IC4.4, IC4.8, Q3.C, R1.2, R20.1, R21.2
- new net VD: BLAST.1, IC4.2, IC4.6, R1.1, R2.2
- net GND: now also C19.1, C3.2, C4.2, IC3.GND, IC4.1, K1.4, K1.S-/R+, Q1.E, Q2.E, Q4.C, R2.1
- net N$45: now also K1.3; no longer C18.-, R16.2, SWITCH.3
- net N$8: now also K1.8; no longer SWITCH.2
- net VA: now also C3.1, IC3.VIN
Other:
- moved on the sheet: BASE, C10, C11, C12, C13, C14, C15, C16, C5, C6, C7, C8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
